File: Hardware/psu.kicad_sch (KiCad schematic)
At the start: 0 parts

Commit message: Schematic completed, started placing
Parts:
- added C4, C5: 10uF, Capacitor_SMD:CP_Elec_6.3x5.7, symbol Device:C_Polarized_Small
- added C6, C7: 22uF, Capacitor_SMD:C_1210_3225Metric, symbol Device:C_Small
- added D2, D3: 1N5819W, Diode_SMD:D_SOD-123, symbol manul_tech:1N5819W
- added L1: 1uH, Inductor_SMD:L_Wuerth_WE-PD2-Typ-MS, symbol Device:L_Small
- added U3: 173950336, manul_tech:SIP3_11.6x8.5mm, symbol manul_tech:173950336
Connections:
- new net: C4.1, D2.1 (K), D3.1 (K), L1.1
- new net: C5.1, L1.2, U3.1 (VIN)
- new net +3V3: C6.1, C7.1, U3.3 (VOUT)
- new net +5V: D2.2 (A)
- new net GND: C4.2, C5.2, C6.2, C7.2, U3.2 (GND)
- new net VBUS: D3.2 (A)

Commit message: completed routing
Parts:
- removed C4, C5: 10uF, Capacitor_SMD:CP_Elec_6.3x5.7, symbol Device:C_Polarized_Small
- removed C6, C7: 22uF, Capacitor_SMD:C_1210_3225Metric, symbol Device:C_Small
- removed D2, D3: 1N5819W, Diode_SMD:D_SOD-123, symbol manul_tech:1N5819W
- removed L1: 1uH, Inductor_SMD:L_Wuerth_WE-PD2-Typ-MS, symbol Device:L_Small
- removed U3: 173950336, manul_tech:SIP3_11.6x8.5mm, symbol manul_tech:173950336
