File: Hardware/sp1_communicator.kicad_sch (KiCad schematic)
At the start: 41 parts, among them J1 615006138421, J2 629722000214, SW1 KSEM31JLFS, SW2 KSEM31JLFS, U1 140357145100, U2 140357145100, U3 173950336, U4 ESP32-C3-WROOM-02U-N4

Commit message: Added missing internal references
Parts:
- D4: MPN (none) -> WS2812C-2020
- D5: MPN (none) -> 150040RS73240; internalRef (none) -> 8.03.007
- L1: internalRef (none) -> 14.00.001
- R2: MPN (none) -> CRCW04021M00DHEDP; internalRef (none) -> 12.02.027
- R3: MPN (none) -> CRCW04021K00DHEDP; internalRef (none) -> 12.02.026
- U1, U2: internalRef (none) -> 8.04.001
- U3: internalRef (none) -> 10.02.001
- U4: value ESP32-C3-WROOM-02U-N4 -> ESP32-C3-WROOM-02-N4; MPN ESP32-C3-WROOM-02U-N4 -> ESP32-C3-WROOM-02-N4; internalRef (none) -> 28.01.007
Changed lines of the file:
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@@
+      (effects (font (size 1.27 1.27)) hide)
+    )
+    (property "MPN" "CRCW04021M00DHEDP" (at 55.88 76.835 0)
+      (effects (font (size 1.27 1.27)) hide)
+    )
+    (property "internalRef" "12.02.027" (at 55.88 76.835 0)
       (effects (font (size 1.27 1.27)) hide)
     )
@@
       (effects (font (size 1.27 1.27)))
     )
+    (property "MPN" "WS2812C-2020" (at 186.69 136.525 0)
+      (effects (font (size 1.27 1.27)) hide)
+    )
     (pin "1")
     (pin "2")
@@
       (effects (font (size 1.27 1.27)) hide)
     )
+    (property "internalRef" "8.04.001" (at 64.77 101.6 0)
+      (effects (font (size 1.27 1.27)) hide)
+    )
     (pin "1")
     (pin "2")
@@
       (effects (font (size 1.27 1.27)) hide)
     )
+    (property "internalRef" "10.02.001" (at 66.04 177.165 0)
+      (effects (font (size 1.27 1.27)) hide)
+    )
     (pin "1")
     (pin "2")
@@
     )
     (property "Datasheet" "~" (at 55.88 96.52 0)
+      (effects (font (size 1.27 1.27)) hide)
+    )
+    (property "MPN" "CRCW04021K00DHEDP" (at 55.88 96.52 0)
+      (effects (font (size 1.27 1.27)) hide)
+    )
+    (property "internalRef" "12.02.026" (at 55.88 96.52 0)
       (effects (font (size 1.27 1.27)) hide)
     )
@@
       (effects (font (size 1.27 1.27)) hide)
     )
+    (property "MPN" "150040RS73240" (at 31.75 180.975 0)
+      (effects (font (size 1.27 1.27)) hide)
+    )
+    (property "internalRef" "8.03.007" (at 31.75 180.975 0)
+      (effects (font (size 1.27 1.27)) hide)
+    )
     (pin "1")
     (pin "2")
@@
     )
     (property "MPN" "7447730" (at 45.72 177.165 90)
+      (effects (font (size 1.27 1.27)) hide)
+    )
+    (property "internalRef" "14.00.001" (at 45.72 177.165 0)
       (effects (font (size 1.27 1.27)) hide)
     )
@@
       (effects (font (size 1.27 1.27)) hide)
     )
+    (property "internalRef" "8.04.001" (at 64.135 72.39 0)
+      (effects (font (size 1.27 1.27)) hide)
+    )
     (pin "1")
     (pin "2")
@@
       (effects (font (size 1.27 1.27)))
     )
-    (property "Value" "ESP32-C3-WROOM-02U-N4" (at 133.35 69.215 0)
+    (property "Value" "ESP32-C3-WROOM-02-N4" (at 133.35 69.215 0)
       (effects (font (size 1.27 1.27)))
     )
@@
       (effects (font (size 1.27 1.27)) hide)
     )
-    (property "MPN" "ESP32-C3-WROOM-02U-N4" (at 133.35 89.535 0)
-      (effects (font (size 1.27 1.27)) hide)
-    )
+    (property "MPN" "ESP32-C3-WROOM-02-N4" (at 133.35 89.535 0)
+      (effects (font (size 1.27 1.27)) hide)
+    )
+    (property "internalRef" "28.01.007" (at 133.35 89.535 0)
+      (effects (font (size 1.27 1.27)) hide)
+    )
