File: Hardware/p1_wireless_indicator.kicad_pcb (KiCad board)
At the start: 4 copper layers, 50.7 x 40 mm, 41 parts, among them J1 615006138421, J2 629722000214, SW1 KSEM31JLFS, SW2 KSEM31JLFS, U1 140357145100, U2 140357145100, U3 173950336, U4 ESP32-C3-WROOM-02U-N4

Commit message: Updated Layout
Parts:
- L1: footprint Inductor_SMD:L_Wuerth_WE-PD2-Typ-MS -> manul_tech:7447730
- U4: value ESP32-C3-WROOM-02U-N4 -> ESP32-C3-WROOM-02-N4
- moved J1 2.09 mm to (97.7, 71.1)
- moved J2 0.77 mm to (137.9, 100.1)
Connections:
- U4 pad 19: GND -> (no net)
- U4 pad 20: GND -> (no net)
- U4 pad 21: GND -> (no net)
- U4 pad 22: GND -> (no net)
- U4 pad 23: GND -> (no net)
- U4 pad 24: GND -> (no net)
- U4 pad 25: GND -> (no net)
- U4 pad 26: GND -> (no net)
- U4 pad 27: GND -> (no net)
- U4 pad 28: GND -> (no net)
- U4 pad 29: GND -> (no net)
- U4 pad 30: GND -> (no net)
- U4 pad 31: GND -> (no net)
- U4 pad 32: GND -> (no net)
- U4 pad 33: GND -> (no net)
- U4 pad 34: GND -> (no net)
- U4 pad 35: GND -> (no net)
- U4 pad 36: GND -> (no net)
- U4 pad 37: GND -> (no net)
- U4 pad 38: GND -> (no net)
- U4 pad 39: GND -> (no net)
Routing:
- net /~{DATA}: track 8.51 -> 10.6 mm
- net /REQ: track 13.1 -> 15.2 mm
- net VBUS: track 49.6 -> 51.3 mm
- net /D-: track 10.6 -> 12.1 mm
- net Net-(J2-CC2): track 4.06 -> 4.83 mm
- net Net-(J2-CC1): track 4.27 -> 5.03 mm
- net /D+: track 7.48 -> 8.25 mm
- net +5V: track 22.4 -> 23.1 mm
Other:
- board text added: "P1 Wireless Interface (P1WI) designed by Manul Technologies 2024 V${REVISION}"
- board text removed: "P1 Wireless Interface (P1WI) designed by Manul Technologies 2024 V1.0"

Commit message: Added 10K resistor on GPIO8 to fix boot issue
Parts:
- added R16: 10K, Resistor_SMD:R_0402_1005Metric, F.Cu at (123.3, 79.1)
Connections:
- U4 pad 7: unconnected-(U4-IO8-Pad7) -> Net-(U4-IO8)
Routing:
- net Net-(U4-IO8): track 0.00 -> 1.66 mm
- net +3V3: track 12.1 -> 13.1 mm, vias 7 -> 8
Changed lines of the file:
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@@
   (net 24 "Net-(R5-Pad2)")
   (net 25 "unconnected-(U4-IO7-Pad6)")
-  (net 26 "unconnected-(U4-IO8-Pad7)")
+  (net 26 "Net-(U4-IO8)")
   (net 27 "unconnected-(U4-IO10-Pad10)")
   (net 28 "unconnected-(U4-RXD{slash}IO20-Pad11)")
@@
       (net 25 "unconnected-(U4-IO7-Pad6)") (pinfunction "IO7") (pintype "bidirectional+no_connect") (solder_mask_margin 0.102))
     (pad "7" smd rect (at -8.75 6.1) (size 1.5 0.9) (layers "F.Cu" "F.Paste" "F.Mask")
-      (net 26 "unconnected-(U4-IO8-Pad7)") (pinfunction "IO8") (pintype "bidirectional+no_connect") (solder_mask_margin 0.102))
+      (net 26 "Net-(U4-IO8)") (pinfunction "IO8") (pintype "bidirectional") (solder_mask_margin 0.102))
     (pad "8" smd rect (at -8.75 7.6) (size 1.5 0.9) (layers "F.Cu" "F.Paste" "F.Mask")
       (net 4 "/BOOT") (pinfunction "IO9") (pintype "bidirectional") (solder_mask_margin 0.102))
@@
     (pad "2" smd roundrect (at 0.51 0 270) (size 0.54 0.64) (layers "F.Cu" "F.Paste" "F.Mask") (roundrect_rratio 0.25)
       (net 24 "Net-(R5-Pad2)") (pintype "passive"))
+    (model "${KICAD6_3DMODEL_DIR}/Resistor_SMD.3dshapes/R_0402_1005Metric.wrl"
+      (offset (xyz 0 0 0))
+      (scale (xyz 1 1 1))
+      (rotate (xyz 0 0 0))
+    )
+  )
+  (footprint "Resistor_SMD:R_0402_1005Metric" (layer "F.Cu")
+    (at 123.27 79.06 -90)
+    (descr "Resistor SMD 0402 (1005 Metric), square (rectangular) end terminal, IPC_7351 nominal, (Body size source: IPC-SM-782 page 72, https://www.pcb-3d.com/wordpress/wp-content/uploads/ipc-sm-782a_amendment_1_and_2.pdf), generated with kicad-footprint-generator")
+    (tags "resistor")
+    (property "MPN" "CRCW040210K0FKEDHP")
+    (property "Sheetfile" "p1_wireless_indicator.kicad_sch")
+    (property "Sheetname" "")
+    (property "internalRef" "12.02.010")
+    (property "ki_description" "Resistor, small symbol")
+    (property "ki_keywords" "R resistor")
+    (attr smd)
+    (fp_text reference "R16" (at -0.26 1.17 90) (layer "F.SilkS")
+        (effects (font (size 1 1) (thickness 0.15)))
+    )
+    (fp_text value "10K" (at 0 1.17 90) (layer "F.Fab")
+        (effects (font (size 1 1) (thickness 0.15)))
+    )
+    (fp_text user "${REFERENCE}" (at 0 0 90) (layer "F.Fab")
+        (effects (font (size 0.26 0.26) (thickness 0.04)))
+    )
+    (fp_line (start -0.153641 -0.38) (end 0.153641 -0.38)
+      (stroke (width 0.12) (type solid)) (layer "F.SilkS"))
+    (fp_line (start -0.153641 0.38) (end 0.153641 0.38)
+      (stroke (width 0.12) (type solid)) (layer "F.SilkS"))
+    (fp_line (start -0.93 -0.47) (end 0.93 -0.47)
+      (stroke (width 0.05) (type solid)) (layer "F.CrtYd"))
+    (fp_line (start -0.93 0.47) (end -0.93 -0.47)
+      (stroke (width 0.05) (type solid)) (layer "F.CrtYd"))
+    (fp_line (start 0.93 -0.47) (end 0.93 0.47)
+      (stroke (width 0.05) (type solid)) (layer "F.CrtYd"))
+    (fp_line (start 0.93 0.47) (end -0.93 0.47)
+      (stroke (width 0.05) (type solid)) (layer "F.CrtYd"))
+    (fp_line (start -0.525 -0.27) (end 0.525 -0.27)
+      (stroke (width 0.1) (type solid)) (layer "F.Fab"))
+    (fp_line (start -0.525 0.27) (end -0.525 -0.27)
+      (stroke (width 0.1) (type solid)) (layer "F.Fab"))
+    (fp_line (start 0.525 -0.27) (end 0.525 0.27)
+      (stroke (width 0.1) (type solid)) (layer "F.Fab"))
+    (fp_line (start 0.525 0.27) (end -0.525 0.27)
+      (stroke (width 0.1) (type solid)) (layer "F.Fab"))
+    (pad "1" smd roundrect (at -0.51 0 270) (size 0.54 0.64) (layers "F.Cu" "F.Paste" "F.Mask") (roundrect_rratio 0.25)
+      (net 1 "+3V3") (pintype "passive"))
+    (pad "2" smd roundrect (at 0.51 0 270) (size 0.54 0.64) (layers "F.Cu" "F.Paste" "F.Mask") (roundrect_rratio 0.25)
+      (net 26 "Net-(U4-IO8)") (pintype "passive"))
     (model "${KICAD6_3DMODEL_DIR}/Resistor_SMD.3dshapes/R_0402_1005Metric.wrl"
       (offset (xyz 0 0 0))
@@
   (segment (start 119.4 71.175) (end 120 70.575) (width 0.125) (layer "F.Cu") (net 1))
   (segment (start 124.925 70.575) (end 121.425 70.575) (width 0.5) (layer "F.Cu") (net 1))
+  (segment (start 123.27 78.55) (end 123.27 77.54) (width 0.125) (layer "F.Cu") (net 1))
   (via (at 128.7 100.5) (size 0.7) (drill 0.35) (layers "F.Cu" "B.Cu") (free) (net 1))
   (via (at 126.7 100.5) (size 0.7) (drill 0.35) (layers "F.Cu" "B.Cu") (free) (net 1))
   (via (at 109 94.725) (size 0.8) (drill 0.4) (layers "F.Cu" "B.Cu") (net 1))
   (via (at 120 70.575) (size 0.7) (drill 0.35) (layers "F.Cu" "B.Cu") (free) (net 1))
+  (via (at 123.27 77.54) (size 0.7) (drill 0.35) (layers "F.Cu" "B.Cu") (net 1))
   (via (at 127.7 100.5) (size 0.7) (drill 0.35) (layers "F.Cu" "B.Cu") (free) (net 1))
   (via (at 127.525 88.43) (size 0.8) (drill 0.4) (layers "F.Cu" "B.Cu") (net 1))
@@
   (segment (start 119.84 77.97) (end 120.725 77.085) (width 0.125) (layer "F.Cu") (net 24))
   (segment (start 118.075 77.97) (end 119.84 77.97) (width 0.125) (layer "F.Cu") (net 24))
+  (segment (start 123.275 79.575) (end 124.925 79.575) (width 0.125) (layer "F.Cu") (net 26))
+  (segment (start 123.27 79.57) (end 123.275 79.575) (width 0.125) (layer "F.Cu") (net 26))
   (segment (start 123.26 69.55) (end 123.26 68.87) (width 0.125) (layer "F.Cu") (net 31))
   (segment (start 122.51 68.12) (end 122.5 68.12) (width 0.125) (layer "F.Cu") (net 31))

Commit message: Rounting of V2.0
Parts:
- removed R2: 1M, Resistor_SMD:R_0402_1005Metric
- added R17: 1M, Resistor_SMD:R_0402_1005Metric, F.Cu at (104.6, 64.3)
- R3: value 1K -> 220R
- U1, U2: footprint Package_SO:SOP-4_3.8x4.1mm_P2.54mm -> manul_tech:140357145100
- moved R10 51.3 mm to (142.5, 70.7), turned to -90 degrees
- moved SW1 50.7 mm to (138.7, 67.2), turned to 90 degrees
- moved J2 43.5 mm to (94.6, 95.4), turned to -90 degrees
- moved C9 42.3 mm to (137.2, 72.8), turned to 180 degrees
- moved SW2 39.3 mm to (130.0, 67.2), turned to 90 degrees
- moved R7 36.3 mm to (104.6, 97.6), turned to 0 degrees
- moved R11 35.0 mm to (132.0, 72.9), turned to -90 degrees
- moved R12 34.8 mm to (140.0, 100.6), turned to 180 degrees
- moved D1 32.8 mm to (105.7, 95.4), turned to 0 degrees
- moved C11 32.7 mm to (108.4, 96.8), turned to -90 degrees
- moved R6 31.2 mm to (104.6, 93.1), turned to 180 degrees
- moved R14 31.1 mm to (110.0, 96.3), turned to 0 degrees
- moved R9 29.2 mm to (132.5, 78.7), turned to 180 degrees
- moved C10 29.1 mm to (108.4, 93.9), turned to 90 degrees
- moved R13 28.6 mm to (110.0, 94.4), turned to 0 degrees
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Connections:
- R4 pad 2: /RX -> Net-(R4-Pad2)
- U2 pad 3: GND -> /RX
- U2 pad 4: /RX -> Net-(R4-Pad2)
Routing:
- net /RTS: track 4.61 -> 51.8 mm, vias 0 -> 2
- net /RX: track 22.1 -> 50.5 mm, vias 2 -> 0
- net VBUS: track 51.3 -> 25.1 mm, vias 4 -> 3
- net Net-(U4-IO2): track 23.9 -> 1.60 mm, vias 2 -> 0
- net /EN: track 37.7 -> 19.6 mm, vias 2 -> 3
- net /DA+: track 11.5 -> 29.0 mm
- net /DA-: track 10.8 -> 28.2 mm
- net /BOOT: track 28.4 -> 13.0 mm, vias 2 -> 0
- net Net-(D2-K): track 14.3 -> 0.00 mm
- net /STATUS_LED: track 12.9 -> 4.26 mm
- net /D-: track 12.1 -> 8.70 mm, vias 2 -> 0
- net +5V: track 23.1 -> 20.2 mm, vias 1 -> 0
- net /D+: track 8.25 -> 9.98 mm, vias 0 -> 2
- net Net-(R4-Pad2): track 0.00 -> 1.60 mm
- net Net-(R5-Pad2): track 3.02 -> 1.62 mm
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Other:
- outline, holes or cut-outs redrawn
